File: crates/sch-layout/tests/snapshots/grid-demo.kicad_sch (KiCad schematic)
At the start: 10 parts, among them U1 NE555P

Commit message: feat(idioms): co-place GPIO LED + series resistor as one vertical leg
Recognize the LED-indicator idiom (an LED in series with a current-limit
resistor) via the graph matcher and tidy it with an mm post-pass: the LED is
report-only (not frozen — normal placement seats it well by the IC pin it taps),
and `align_led_chains` (in emit, on FINAL positions like align_idiom_clusters)
snaps the resistor into a clean vertical leg directly below the LED, re-orienting
both vertical so they read as one collinear GPIO -> LED -> R -> GND string instead
of the resistor scattering to a spare column with a long node wire.

Why report-only + post-pass rather than a frozen pre-placement: a GPIO LED taps
its IC on the same edge as the crystal, so a frozen chain there collides with the
crystal cluster and (being frozen) forces other parts onto the IC text. Running on
final positions sidesteps the grid's lack of idiom-region allocation, and the
follow-up decongest nudges anything the moved resistor overlaps.

Idiom gains a `freeze` flag (crystal/decoupling freeze + seed cells; led_indicator
reports only). Resolves the LED-scatter critic major on the STM32 fixture (0
warnings); grid-demo re-blessed (its 555 indicator now a clean leg). Greedy netlist
oracle green on all fixtures.

Co-Authored-By: Claude Opus 4.8 (1M context) <noreply@anthropic.com>
Connections:
- net GND: now also D1.2 (A), R3.2
Other:
- moved on the sheet: D1, J2, R3
Changed lines of the file:
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@@
 	(generator "auto-pcb")
 	(generator_version "0.1")
-	(paper "User" 120.64999999999999 96.52000000000001)
+	(paper "User" 120.64999999999999 102.87)
 	(title_block
 		(title "grid-demo")
@@
 	(wire
 		(pts
-			(xy 66.04 33.02) (xy 71.12 33.02)
+			(xy 66.04 33.02) (xy 80.01 33.02)
 		)
 		(stroke (width 0) (type default))
@@
 	(wire
 		(pts
-			(xy 71.12 33.02) (xy 71.12 27.939999999999998)
-		)
-		(stroke (width 0) (type default))
-	)
-	(wire
-		(pts
-			(xy 71.12 33.02) (xy 80.01 33.02)
-		)
-		(stroke (width 0) (type default))
-	)
-	(wire
-		(pts
-			(xy 77.47 57.15) (xy 77.47 78.74000000000001)
+			(xy 74.93 53.339999999999996) (xy 74.93 87.63000000000001)
+		)
+		(stroke (width 0) (type default))
+	)
+	(wire
+		(pts
+			(xy 74.93 87.63000000000001) (xy 87.63 87.63000000000001)
+		)
+		(stroke (width 0) (type default))
+	)
+	(wire
+		(pts
+			(xy 77.47 55.88) (xy 77.47 78.74000000000001)
 		)
 		(stroke (width 0) (type default))
@@
 	(wire
 		(pts
-			(xy 78.74 27.939999999999998) (xy 87.63 27.939999999999998)
-		)
-		(stroke (width 0) (type default))
-	)
-	(wire
-		(pts
-			(xy 80.01 33.02) (xy 80.01 54.61)
-		)
-		(stroke (width 0) (type default))
-	)
-	(wire
-		(pts
-			(xy 80.01 57.15) (xy 77.47 57.15)
-		)
-		(stroke (width 0) (type default))
-	)
-	(wire
-		(pts
-			(xy 87.63 27.939999999999998) (xy 87.63 66.04)
-		)
-		(stroke (width 0) (type default))
-	)
-	(wire
-		(pts
-			(xy 87.63 73.66000000000001) (xy 87.63 78.74000000000001)
+			(xy 80.01 33.02) (xy 80.01 53.339999999999996)
+		)
+		(stroke (width 0) (type default))
+	)
+	(wire
+		(pts
+			(xy 80.01 53.339999999999996) (xy 74.93 53.339999999999996)
+		)
+		(stroke (width 0) (type default))
+	)
+	(wire
+		(pts
+			(xy 80.01 55.88) (xy 77.47 55.88)
+		)
+		(stroke (width 0) (type default))
+	)
+	(wire
+		(pts
+			(xy 87.63 63.5) (xy 87.63 71.12)
+		)
+		(stroke (width 0) (type default))
+	)
+	(wire
+		(pts
+			(xy 87.63 71.12) (xy 87.63 78.74000000000001)
+		)
+		(stroke (width 0) (type default))
+	)
+	(wire
+		(pts
+			(xy 87.63 78.74000000000001) (xy 87.63 80.01)
 		)
 		(stroke (width 0) (type default))
@@
 	)
 	(junction
-		(at 66.04 33.02)
-		(diameter 0)
-		(color 0 0 0 0)
-	)
-	(junction
 		(at 66.04 43.18)
 		(diameter 0)
@@
 	)
 	(junction
-		(at 71.12 33.02)
+		(at 74.93 53.339999999999996)
+		(diameter 0)
+		(color 0 0 0 0)
+	)
+	(junction
+		(at 74.93 87.63000000000001)
 		(diameter 0)
 		(color 0 0 0 0)
@@
 	)
 	(junction
-		(at 87.63 27.939999999999998)
+		(at 80.01 53.339999999999996)
 		(diameter 0)
 		(color 0 0 0 0)
@@
 	(symbol
 		(lib_id "Device:LED")
-		(at 87.63 69.85000000000001 90)
+		(at 87.63 67.31 270)
 		(unit 1)
 		(exclude_from_sim no)
@@
 		(dnp no)
 		(property "Reference" "D1"
-			(at 93.98 68.58 270)
+			(at 93.98 66.04 90)
 			(effects (font (size 1.27 1.27)) (justify left))
 		)
 		(property "Value" "red"
-			(at 93.98 71.12 270)
-			(effects (font (size 1.27 1.27)) (justify left))
-		)
-		(property "Footprint" ""
-			(at 87.63 69.85000000000001 0)
+			(at 93.98 68.58 90)
+			(effects (font (size 1.27 1.27)) (justify left))
+		)
+		(property "Footprint" ""
+			(at 87.63 67.31 0)
 			(effects (font (size 1.27 1.27)) (hide yes))
 		)
@@
 	(symbol
 		(lib_id "Connector_Generic:Conn_01x02")
-		(at 85.09 54.61 0)
+		(at 85.09 53.339999999999996 0)
 		(unit 1)
 		(exclude_from_sim no)
@@
 		(dnp no)
 		(property "Reference" "J2"
-			(at 91.44 53.34 0)
+			(at 91.44 52.07 0)
 			(effects (font (size 1.27 1.27)) (justify left))
 		)
 		(property "Value" ""
-			(at 91.44 55.88 0)
-			(effects (font (size 1.27 1.27)) (justify left))
-		)
-		(property "Footprint" ""
-			(at 85.09 54.61 0)
+			(at 91.44 54.61 0)
+			(effects (font (size 1.27 1.27)) (justify left))
+		)
+		(property "Footprint" ""
+			(at 85.09 53.339999999999996 0)
 			(effects (font (size 1.27 1.27)) (hide yes))
 		)
@@
 	(symbol
 		(lib_id "Device:R")
-		(at 74.93 27.939999999999998 90)
+		(at 87.63 83.82000000000001 180)
 		(unit 1)
 		(exclude_from_sim no)
@@
 		(dnp no)
 		(property "Reference" "R3"
-			(at 74.93 35.26 270)
-			(effects (font (size 1.27 1.27)))
+			(at 93.98 82.55 0)
+			(effects (font (size 1.27 1.27)) (justify left))
 		)
 		(property "Value" "1k"
-			(at 74.93 37.8 270)
-			(effects (font (size 1.27 1.27)))
-		)
-		(property "Footprint" ""
-			(at 74.93 27.939999999999998 0)
-			(effects (font (size 1.27 1.27)) (hide yes))
-		)
+			(at 93.98 85.09 0)
+			(effects (font (size 1.27 1.27)) (justify left))
+		)
+		(property "Footprint" ""
+			(at 87.63 83.82000000000001 0)
+			(effects (font (size 1.27 1.27)) (hide yes))
+		)
